Commit message: Added inertials

File: urdf/fr3.urdf (robot description, URDF)
Before this commit: robot fr3, 13 links, 12 joints
Links:
- link fr3_hand: mass None -> 0.6544
- link fr3_leftfinger: mass None -> 0.0291
- link fr3_link0: mass None -> 2.3966
- link fr3_link1: mass None -> 2.9274653454
- link fr3_link2: mass None -> 2.9355370338
- link fr3_link3: mass None -> 2.2449013699
- link fr3_link4: mass None -> 2.6155955791
- link fr3_link5: mass None -> 2.3271207594
- link fr3_link6: mass None -> 1.8170376524
- link fr3_link7: mass None -> 0.6271432862
- link fr3_link_stationary: mass None -> 5.500
- link fr3_rightfinger: mass None -> 0.0291

Commit message: linear platform tuning - incomplete

File: urdf/fr3.urdf (robot description, URDF)
Before this commit: robot fr3, 13 links, 12 joints
Joints:
- joint fr3_joint_linear: limit lower=0.0 upper=0.72 effort=87.0 velocity=0.5 -> lower=0.0 upper=0.72 effort=200.0 velocity=0.75
